File: rp2c02-rp2040/rp2c02-rp2040.kicad_pcb (KiCad board)
At the start: 2 copper layers, 96.5 x 63.5 mm, 25 parts, among them J1 VIDEO, J2 Si5351A, Q1 2SA937, Q2 AO3400A, SW1 RUN, U1 RP2C02, U2 74HC574N, U3 IS62C256AL, U4 Pico

Commit message: レベルシフト版/レベルシフト基板追加、通常基板の2SA937ピン逆転修正
Connections:
- Q1 pad 1: GND -> Net-(Q1-E)
- Q1 pad 2: Net-(Q1-C) -> GND
- R1 pad 2: Net-(Q1-C) -> Net-(Q1-E)
- R2 pad 1: Net-(Q1-C) -> Net-(Q1-E)
Routing:
- net Net-(Q1-E): track 0.00 -> 15.7 mm
- net Net-(Q1-C): track 15.2 -> 0.00 mm
Other:
- board text added: "C02:J:A:A:2024092600"
- board text added: "VCC"
- board text added: "w/RP2040 rev.1.1 by DJ KUR4GE"
- board text removed: "C02:J:A:A:2024091300"
- board text removed: "w/RP2040 rev.1 by DJ KUR4GE"

Commit message: 74HC573に修正
Parts:
- U2: value 74HC574N -> 74HC573N
Other:
- board text added: "74HC573"
- board text removed: "74HC574"
Changed lines of the file:
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@@
 			)
 		)
-		(property "Value" "74HC574N"
+		(property "Value" "74HC573N"
 			(at 3.81 25.19 0)
 			(layer "F.Fab")
@@
 			)
 		)
-		(property "Datasheet" "http://www.ti.com/lit/gpn/sn74LS574"
+		(property "Datasheet" "74xx/74hc573.pdf"
 			(at 0 0 0)
 			(unlocked yes)
@@
 			)
 		)
-		(property "Description" "8-bit Register, 3-state outputs"
+		(property "Description" "8-bit Latch 3-state outputs"
 			(at 0 0 0)
 			(unlocked yes)
@@
 			(remove_unused_layers no)
 			(net 27 "/P.ALE")
-			(pinfunction "Cp")
+			(pinfunction "Load")
 			(pintype "input")
 		)
@@
 		)
 	)
-	(gr_text "74HC574"
+	(gr_text "74HC573"
 		(at 127.635 76.2 90)
 		(layer "F.SilkS")
